File: board/ft2232_submod.sch (KiCad schematic (older format))
At the start: 24 parts, among them U1 FT2232H-56, U2 93LC46B, Y1 12.000MHz

Commit message: Update for release.
Parts:
- C1, C4: Comment (none) -> Substitution Okay; Digikey (none) -> 1276-1183-1-ND
- C10, C11, C12, C13, C2, C5, C8, C9: Comment (none) -> Substitution Okay; Digikey (none) -> 1276-1857-1-ND
- C3: Comment (none) -> Substitution Okay; Digikey (none) -> 1276-1892-1-ND; P/N GRM188R61A335KE15D -> CL10A335KP8NNNC
- C6, C7: Digikey (none) -> 311-1063-1-ND; P/N VJ0603A270JXACW1BC -> CC0603JRNPO9BN270
- FB1, FB2: Digikey (none) -> 445-1567-1-ND
- R1: Digikey (none) -> RMCF0603FT12K0CT-ND
- R2, R3, R4, R6: Comment (none) -> Substitution Okay; Digikey (none) -> RMCF0603JT10K0CT-ND
- R5: Comment (none) -> Substitution Okay; Digikey (none) -> RMCF0603JT2K20CT-ND
- U1: Digikey (none) -> 768-1276-ND
- U2: Digikey (none) -> 93LC46BT-I/SNCT-ND
- Y1: Digikey (none) -> 535-15006-1-ND; P/N FOXSDLF/120-20/TR -> ABLS-12.000MHZ-20-B-3-H-T
Changed lines of the file:
@@
 EESchema Schematic File Version 4
-LIBS:board-cache
 EELAYER 30 0
 EELAYER END
@@
 encoding utf-8
 Sheet 2 3
-Title "Universal IoT Interface"
-Date "2019-06-23"
-Rev "Rev 3"
-Comp "Matir / systemoverlord.com"
-Comment1 "Copyright 2019 Google, LLC"
-Comment2 ""
+Title "Test Interface for Multiple Embedded Protocols"
+Date "2020-05-08"
+Rev "Rev 5"
+Comp "Copyright 2020 Google, LLC"
+Comment1 "Designer: @Matir / systemoverlord.com"
+Comment2 "License: Apache2"
 Comment3 ""
 Comment4 ""
@@
 F 3 "" H 6350 3450 50  0001 C CNN
 F 4 "FT2232H-56Q-TRAY" H 0   0   50  0001 C CNN "P/N"
+F 5 "768-1276-ND" H 5650 3500 50  0001 C CNN "Digikey"
 	1    5650 3500
 	1    0    0    -1
@@
 F 2 "Capacitor_SMD:C_0603_1608Metric" H 3450 2000 50  0001 C CNN
 F 3 "~" H 3450 2000 50  0001 C CNN
-F 4 "GRM188R61A335KE15D" H 0   0   50  0001 C CNN "P/N"
+F 4 "CL10A335KP8NNNC" H 0   0   50  0001 C CNN "P/N"
+F 5 "Substitution Okay" H 3450 2000 50  0001 C CNN "Comment"
+F 6 "1276-1892-1-ND" H 3450 2000 50  0001 C CNN "Digikey"
 	1    3450 2000
 	1    0    0    -1
@@
 F 3 "~" H 4000 2600 50  0001 C CNN
 F 4 "RMCF0603FT12K0" H 0   0   50  0001 C CNN "P/N"
+F 5 "RMCF0603FT12K0CT-ND" H 4000 2600 50  0001 C CNN "Digikey"
 	1    4000 2600
 	0    1    1    0
@@
 F 3 "~" H 3650 900 50  0001 C CNN
 F 4 "MPZ2012S101AT000" H 0   0   50  0001 C CNN "P/N"
+F 5 "445-1567-1-ND" H 3650 900 50  0001 C CNN "Digikey"
 	1    3650 900
 	1    0    0    -1
@@
 F 3 "~" H 3300 900 50  0001 C CNN
 F 4 "MPZ2012S101AT000" H 0   0   50  0001 C CNN "P/N"
+F 5 "445-1567-1-ND" H 3300 900 50  0001 C CNN "Digikey"
 	1    3300 900
 	1    0    0    -1
@@
 F 3 "~" H 3650 1300 50  0001 C CNN
 F 4 "CL10A225KQ8NNNC" H 0   0   50  0001 C CNN "P/N"
+F 5 "Substitution Okay" H 3650 1300 50  0001 C CNN "Comment"
+F 6 "1276-1183-1-ND" H 3650 1300 50  0001 C CNN "Digikey"
 	1    3650 1300
 	1    0    0    -1
@@
 F 3 "~" H 3300 1300 50  0001 C CNN
 F 4 "CL10A104KA8NNNC" H 0   0   50  0001 C CNN "P/N"
+F 5 "Substitution Okay" H 3300 1300 50  0001 C CNN "Comment"
+F 6 "1276-1857-1-ND" H 3300 1300 50  0001 C CNN "Digikey"
 	1    3300 1300
 	1    0    0    -1
@@
 F 3 "~" H 3900 1300 50  0001 C CNN
 F 4 "CL10A104KA8NNNC" H 0   0   50  0001 C CNN "P/N"
+F 5 "Substitution Okay" H 3900 1300 50  0001 C CNN "Comment"
+F 6 "1276-1857-1-ND" H 3900 1300 50  0001 C CNN "Digikey"
 	1    3900 1300
 	1    0    0    -1
@@
 F 3 "~" H 3050 1300 50  0001 C CNN
 F 4 "CL10A225KQ8NNNC" H 0   0   50  0001 C CNN "P/N"
+F 5 "Substitution Okay" H 3050 1300 50  0001 C CNN "Comment"
+F 6 "1276-1183-1-ND" H 3050 1300 50  0001 C CNN "Digikey"
 	1    3050 1300
 	1    0    0    -1
@@
 F 3 "~" H 8600 1300 50  0001 C CNN
 F 4 "CL10A104KA8NNNC" H 0   0   50  0001 C CNN "P/N"
+F 5 "Substitution Okay" H 8600 1300 50  0001 C CNN "Comment"
+F 6 "1276-1857-1-ND" H 8600 1300 50  0001 C CNN "Digikey"
 	1    8600 1300
 	1    0    0    -1
@@
 F 3 "~" H 9000 1300 50  0001 C CNN
 F 4 "CL10A104KA8NNNC" H 0   0   50  0001 C CNN "P/N"
+F 5 "Substitution Okay" H 9000 1300 50  0001 C CNN "Comment"
+F 6 "1276-1857-1-ND" H 9000 1300 50  0001 C CNN "Digikey"
 	1    9000 1300
 	1    0    0    -1
@@
 F 3 "~" H 9400 1300 50  0001 C CNN
 F 4 "CL10A104KA8NNNC" H 0   0   50  0001 C CNN "P/N"
+F 5 "Substitution Okay" H 9400 1300 50  0001 C CNN "Comment"
+F 6 "1276-1857-1-ND" H 9400 1300 50  0001 C CNN "Digikey"
 	1    9400 1300
 	1    0    0    -1
@@
 F 3 "~" H 9800 1300 50  0001 C CNN
 F 4 "CL10A104KA8NNNC" H 0   0   50  0001 C CNN "P/N"
+F 5 "Substitution Okay" H 9800 1300 50  0001 C CNN "Comment"
+F 6 "1276-1857-1-ND" H 9800 1300 50  0001 C CNN "Digikey"
 	1    9800 1300
 	1    0    0    -1
@@
 F 3 "~" H 10200 1300 50  0001 C CNN
 F 4 "CL10A104KA8NNNC" H 0   0   50  0001 C CNN "P/N"
+F 5 "Substitution Okay" H 10200 1300 50  0001 C CNN "Comment"
+F 6 "1276-1857-1-ND" H 10200 1300 50  0001 C CNN "Digikey"
 	1    10200 1300
 	1    0    0    -1
@@
 F 3 "~" H 4000 2900 50  0001 C CNN
 F 4 "RMCF0603JT10K0" H 0   0   50  0001 C CNN "P/N"
+F 5 "Substitution Okay" H 4000 2900 50  0001 C CNN "Comment"
+F 6 "RMCF0603JT10K0CT-ND" H 4000 2900 50  0001 C CNN "Digikey"
 	1    4000 2900
 	0    1    1    0
@@
 F 2 "Crystal:Crystal_SMD_HC49-SD" H 1850 3250 50  0001 C CNN
 F 3 "~" H 1850 3250 50  0001 C CNN
-F 4 "FOXSDLF/120-20/TR" H 0   0   50  0001 C CNN "P/N"
+F 4 "ABLS-12.000MHZ-20-B-3-H-T" H 0   0   50  0001 C CNN "P/N"
+F 5 "535-15006-1-ND" H 1850 3250 50  0001 C CNN "Digikey"
 	1    1850 3250
 	1    0    0    -1
@@
 F 2 "Capacitor_SMD:C_0603_1608Metric" H 2200 3500 50  0001 C CNN
 F 3 "~" H 2200 3500 50  0001 C CNN
-F 4 "VJ0603A270JXACW1BC" H 0   0   50  0001 C CNN "P/N"
+F 4 "CC0603JRNPO9BN270" H 0   0   50  0001 C CNN "P/N"
+F 5 "311-1063-1-ND" H 2200 3500 50  0001 C CNN "Digikey"
 	1    2200 3500
 	1    0    0    -1
@@
 F 2 "Capacitor_SMD:C_0603_1608Metric" H 1500 3500 50  0001 C CNN
 F 3 "~" H 1500 3500 50  0001 C CNN
-F 4 "VJ0603A270JXACW1BC" H 0   0   50  0001 C CNN "P/N"
+F 4 "CC0603JRNPO9BN270" H 0   0   50  0001 C CNN "P/N"
+F 5 "311-1063-1-ND" H 1500 3500 50  0001 C CNN "Digikey"
 	1    1500 3500
 	1    0    0    -1
@@
 F 3 "http://ww1.microchip.com/downloads/en/DeviceDoc/20001749K.pdf" H 2000 5700 50  0001 C CNN
 F 4 "93LC46BT-I/SN" H 0   0   50  0001 C CNN "P/N"
+F 5 "93LC46BT-I/SNCT-ND" H 2000 5700 50  0001 C CNN "Digikey"
 	1    2000 5700
 	1    0    0    -1
@@
 F 3 "~" H 3350 5300 50  0001 C CNN
 F 4 "CL10A104KA8NNNC" H 0   0   50  0001 C CNN "P/N"
+F 5 "Substitution Okay" H 3350 5300 50  0001 C CNN "Comment"
+F 6 "1276-1857-1-ND" H 3350 5300 50  0001 C CNN "Digikey"
 	1    3350 5300
 	1    0    0    -1
@@
 F 3 "~" H 2600 5350 50  0001 C CNN
 F 4 "RMCF0603JT10K0" H 0   0   50  0001 C CNN "P/N"
+F 5 "Substitution Okay" H 2600 5350 50  0001 C CNN "Comment"
+F 6 "RMCF0603JT10K0CT-ND" H 2600 5350 50  0001 C CNN "Digikey"
 	1    2600 5350
 	1    0    0    -1
@@
 F 3 "~" H 2850 5350 50  0001 C CNN
 F 4 "RMCF0603JT10K0" H 0   0   50  0001 C CNN "P/N"
+F 5 "Substitution Okay" H 2850 5350 50  0001 C CNN "Comment"
+F 6 "RMCF0603JT10K0CT-ND" H 2850 5350 50  0001 C CNN "Digikey"
 	1    2850 5350
 	1    0    0    -1
@@
 F 3 "~" H 1500 5350 50  0001 C CNN
 F 4 "RMCF0603JT10K0" H 0   0   50  0001 C CNN "P/N"
+F 5 "Substitution Okay" H 1500 5350 50  0001 C CNN "Comment"
+F 6 "RMCF0603JT10K0CT-ND" H 1500 5350 50  0001 C CNN "Digikey"
 	1    1500 5350
 	1    0    0    -1
@@
 F 3 "~" H 2750 5800 50  0001 C CNN
 F 4 "RMCF0603JT2K20" H 0   0   50  0001 C CNN "P/N"
+F 5 "Substitution Okay" H 2750 5800 50  0001 C CNN "Comment"
+F 6 "RMCF0603JT2K20CT-ND" H 2750 5800 50  0001 C CNN "Digikey"
 	1    2750 5800
 	0    1    1    0
