File: board/power.sch (KiCad schematic (older format))
At the start: 22 parts, among them SW1 SW_DP3T, SW2 SW_DP3T, U3 AP2112K-3.3, U4 AP2112K-1.8

Commit message: Update for release.
Parts:
- C14, C15, C16, C17: Comment (none) -> Substitution Okay; Digikey (none) -> 1276-1892-1-ND; P/N CL10A225KQ8NNNC -> CL10A335KP8NNNC
- D7, D8, D9: Comment (none) -> Substitution Okay; Digikey (none) -> 732-4979-1-ND; P/N (none) -> 150060SS75000
- R18, R19, R20: Comment (none) -> Substitution Okay; Digikey (none) -> RMCF0603JT1K00CT-ND; P/N (none) -> RMCF0603JT1K00
- SW1, SW2: Digikey (none) -> CKN10849CT-ND; P/N (none) -> JS203011SCQN
- TPGND2: Comment (none) -> No Populate
- U3: Digikey (none) -> AP2112K-3.3TRG1DICT-ND; P/N (none) -> AP2112K-3.3TRG1
- U4: Digikey (none) -> AP2112K-1.8TRG1DICT-ND; P/N (none) -> AP2112K-1.8TRG1
Changed lines of the file:
@@
 EESchema Schematic File Version 4
-LIBS:board-cache
 EELAYER 30 0
 EELAYER END
@@
 encoding utf-8
 Sheet 3 3
-Title "Universal IoT Interface"
-Date "2019-06-23"
-Rev "Rev 3"
-Comp "Matir / systemoverlord.com"
-Comment1 "Copyright 2019 Google, LLC"
-Comment2 ""
+Title "Test Interface for Multiple Embedded Protocols"
+Date "2020-05-08"
+Rev "Rev 5"
+Comp "Copyright 2020 Google, LLC"
+Comment1 "Designer: @Matir / systemoverlord.com"
+Comment2 "License: Apache2"
 Comment3 ""
 Comment4 ""
@@
 F 2 "Capacitor_SMD:C_0603_1608Metric" H 3100 2200 50  0001 C CNN
 F 3 "~" H 3100 2200 50  0001 C CNN
-F 4 "CL10A225KQ8NNNC" H 650 -450 50  0001 C CNN "P/N"
+F 4 "CL10A335KP8NNNC" H 650 -450 50  0001 C CNN "P/N"
+F 5 "Substitution Okay" H 3100 2200 50  0001 C CNN "Comment"
+F 6 "1276-1892-1-ND" H 3100 2200 50  0001 C CNN "Digikey"
 	1    3100 2200
 	1    0    0    -1
@@
 F 2 "Capacitor_SMD:C_0603_1608Metric" H 1800 2200 50  0001 C CNN
 F 3 "~" H 1800 2200 50  0001 C CNN
-F 4 "CL10A225KQ8NNNC" H 650 -450 50  0001 C CNN "P/N"
+F 4 "CL10A335KP8NNNC" H 650 -450 50  0001 C CNN "P/N"
+F 5 "Substitution Okay" H 1800 2200 50  0001 C CNN "Comment"
+F 6 "1276-1892-1-ND" H 1800 2200 50  0001 C CNN "Digikey"
 	1    1800 2200
 	1    0    0    -1
@@
 F 2 "Capacitor_SMD:C_0603_1608Metric" H 1800 3250 50  0001 C CNN
 F 3 "~" H 1800 3250 50  0001 C CNN
-F 4 "CL10A225KQ8NNNC" H 650 -450 50  0001 C CNN "P/N"
+F 4 "CL10A335KP8NNNC" H 650 -450 50  0001 C CNN "P/N"
+F 5 "Substitution Okay" H 1800 3250 50  0001 C CNN "Comment"
+F 6 "1276-1892-1-ND" H 1800 3250 50  0001 C CNN "Digikey"
 	1    1800 3250
 	1    0    0    -1
@@
 F 2 "Capacitor_SMD:C_0603_1608Metric" H 3100 3250 50  0001 C CNN
 F 3 "~" H 3100 3250 50  0001 C CNN
-F 4 "CL10A225KQ8NNNC" H 650 -450 50  0001 C CNN "P/N"
+F 4 "CL10A335KP8NNNC" H 650 -450 50  0001 C CNN "P/N"
+F 5 "Substitution Okay" H 3100 3250 50  0001 C CNN "Comment"
+F 6 "1276-1892-1-ND" H 3100 3250 50  0001 C CNN "Digikey"
 	1    3100 3250
 	1    0    0    -1
@@
 F 2 "Package_TO_SOT_SMD:SOT-23-5" H 2450 2425 50  0001 C CNN
 F 3 "https://www.diodes.com/assets/Datasheets/AP2112.pdf" H 2450 2200 50  0001 C CNN
+F 4 "AP2112K-3.3TRG1DICT-ND" H 2450 2100 50  0001 C CNN "Digikey"
+F 5 "AP2112K-3.3TRG1" H 2450 2100 50  0001 C CNN "P/N"
 	1    2450 2100
 	1    0    0    -1
@@
 F 2 "Package_TO_SOT_SMD:SOT-23-5" H 2450 3475 50  0001 C CNN
 F 3 "https://www.diodes.com/assets/Datasheets/AP2112.pdf" H 2450 3250 50  0001 C CNN
+F 4 "AP2112K-1.8TRG1DICT-ND" H 2450 3150 50  0001 C CNN "Digikey"
+F 5 "AP2112K-1.8TRG1" H 2450 3150 50  0001 C CNN "P/N"
 	1    2450 3150
 	1    0    0    -1
@@
 F 2 "Matir_Parts:JS203011SCQN" H 5250 1800 50  0001 C CNN
 F 3 "" H 5250 1800 50  0001 C CNN
+F 4 "CKN10849CT-ND" H 5250 2100 50  0001 C CNN "Digikey"
+F 5 "JS203011SCQN" H 5250 2100 50  0001 C CNN "P/N"
 	1    5250 2100
 	1    0    0    -1
@@
 F 2 "Resistor_SMD:R_0603_1608Metric" H 5550 2600 50  0001 C CNN
 F 3 "~" H 5550 2600 50  0001 C CNN
+F 4 "Substitution Okay" H 5550 2600 50  0001 C CNN "Comment"
+F 5 "RMCF0603JT1K00CT-ND" H 5550 2600 50  0001 C CNN "Digikey"
+F 6 "RMCF0603JT1K00" H 5550 2600 50  0001 C CNN "P/N"
 	1    5550 2600
 	1    0    0    -1
@@
 F 2 "Resistor_SMD:R_0603_1608Metric" H 5800 2600 50  0001 C CNN
 F 3 "~" H 5800 2600 50  0001 C CNN
+F 4 "Substitution Okay" H 5800 2600 50  0001 C CNN "Comment"
+F 5 "RMCF0603JT1K00CT-ND" H 5800 2600 50  0001 C CNN "Digikey"
+F 6 "RMCF0603JT1K00" H 5800 2600 50  0001 C CNN "P/N"
 	1    5800 2600
 	1    0    0    -1
@@
 F 2 "Resistor_SMD:R_0603_1608Metric" H 6050 2600 50  0001 C CNN
 F 3 "~" H 6050 2600 50  0001 C CNN
+F 4 "Substitution Okay" H 6050 2600 50  0001 C CNN "Comment"
+F 5 "RMCF0603JT1K00CT-ND" H 6050 2600 50  0001 C CNN "Digikey"
+F 6 "RMCF0603JT1K00" H 6050 2600 50  0001 C CNN "P/N"
 	1    6050 2600
 	1    0    0    -1
@@
 F 2 "LED_SMD:LED_0603_1608Metric" H 5550 2950 50  0001 C CNN
 F 3 "~" H 5550 2950 50  0001 C CNN
+F 4 "Substitution Okay" H 5550 2950 50  0001 C CNN "Comment"
+F 5 "732-4979-1-ND" H 5550 2950 50  0001 C CNN "Digikey"
+F 6 "150060SS75000" H 5550 2950 50  0001 C CNN "P/N"
 	1    5550 2950
 	0    -1   -1   0
@@
 F 2 "LED_SMD:LED_0603_1608Metric" H 5800 2950 50  0001 C CNN
 F 3 "~" H 5800 2950 50  0001 C CNN
+F 4 "Substitution Okay" H 5800 2950 50  0001 C CNN "Comment"
+F 5 "732-4979-1-ND" H 5800 2950 50  0001 C CNN "Digikey"
+F 6 "150060SS75000" H 5800 2950 50  0001 C CNN "P/N"
 	1    5800 2950
 	0    -1   -1   0
@@
 F 2 "LED_SMD:LED_0603_1608Metric" H 6050 2950 50  0001 C CNN
 F 3 "~" H 6050 2950 50  0001 C CNN
+F 4 "Substitution Okay" H 6050 2950 50  0001 C CNN "Comment"
+F 5 "732-4979-1-ND" H 6050 2950 50  0001 C CNN "Digikey"
+F 6 "150060SS75000" H 6050 2950 50  0001 C CNN "P/N"
 	1    6050 2950
 	0    -1   -1   0
@@
 F 2 "Matir_Parts:JS203011SCQN" H 7600 1800 50  0001 C CNN
 F 3 "" H 7600 1800 50  0001 C CNN
+F 4 "CKN10849CT-ND" H 7600 2100 50  0001 C CNN "Digikey"
+F 5 "JS203011SCQN" H 7600 2100 50  0001 C CNN "P/N"
 	1    7600 2100
 	1    0    0    -1
@@
 F 2 "Connector_PinHeader_2.54mm:PinHeader_1x01_P2.54mm_Vertical" H 1050 3800 50  0001 C CNN
 F 3 "~" H 1050 3800 50  0001 C CNN
+F 4 "No Populate" H 850 3800 50  0001 C CNN "Comment"
 	1    850  3800
 	1    0    0    -1
